File: esp32.kicad_sch (KiCad schematic)
At the start: 21 parts, among them J2 TC2030-IDC, J3 Conn_01x04, J4 Conn_01x06, J5 USB_C_Receptacle_USB2.0, SW1 GT-TC029B-H025-L1N, SW2 GT-TC029B-H025-L1N, U3 RT9080-33GJ5, U4 ESP32-S3-WROOM-1

Commit message: added files for model 605 Gamma Kit
Updated sizes for handsoldering kit, added onboard ethernet, cpu heatsink footprint, updated power supply
Parts:
- removed J4: Conn_01x06, Connector_PinHeader_2.54mm:PinHeader_1x06_P2.54mm_Vertical, symbol Connector_Generic:Conn_01x06
- removed J5: USB_C_Receptacle_USB2.0, bitaxe:USB_C_Receptacle_GCT_USB4105-xx-A, symbol bitaxe:USB_C_Receptacle_USB2.0
- removed SW1, SW2: GT-TC029B-H025-L1N, bitaxe:SW_CS1213AGF260_CRS, symbol bitaxe:GT-TC029B-H025-L1N
- removed U3: RT9080-33GJ5, bitaxe:RT9080-33GJ5, symbol bitaxe:RT9080-33GJ5
- added C70, C80: 10nF, Capacitor_SMD:C_0805_2012Metric_Pad1.18x1.45mm_HandSolder, symbol Device:C
- added C71: 4.7uF, Capacitor_SMD:C_0805_2012Metric_Pad1.18x1.45mm_HandSolder, symbol Device:C
- added C72: 1uF, Capacitor_SMD:C_0805_2012Metric_Pad1.18x1.45mm_HandSolder, symbol Device:C
- added C73, C75: .01, Capacitor_SMD:C_0805_2012Metric_Pad1.18x1.45mm_HandSolder, symbol Device:C
- added C74: 22uF, Capacitor_SMD:C_1210_3225Metric_Pad1.33x2.70mm_HandSolder, symbol Device:C
- added C76: 22nF, Capacitor_SMD:C_0805_2012Metric_Pad1.18x1.45mm_HandSolder, symbol Device:C
- added C77: 1nF, Capacitor_SMD:C_0805_2012Metric_Pad1.18x1.45mm_HandSolder, symbol Device:C
- added C78, C79: 6800pF, Capacitor_SMD:C_0805_2012Metric_Pad1.18x1.45mm_HandSolder, symbol Device:C
- added J10: Front PWR / ACT, bitaxe:TE_5-146280-5, symbol Connector:Conn_01x05_Pin
- added J11: EXT Display, bitaxe:TE_5-146280-5, symbol Connector:Conn_01x05_Pin
- added J4: RJ45_Amphenol_RJMG1BD3B8K1ANR, Connector_RJ:RJ45_Amphenol_RJMG1BD3B8K1ANR, symbol Connector:RJ45_Amphenol_RJMG1BD3B8K1ANR
- added J8: USB Header, bitaxe:TE_5-146280-5, symbol Connector:Conn_01x05_Pin
- added J9: Front Controls, bitaxe:TE_5-146280-5, symbol Connector:Conn_01x05_Pin
- added R30: 23.2k, PCM_Resistor_SMD_AKL:R_0805_2012Metric, symbol Device:R_US
- added R31: 13.3k, PCM_Resistor_SMD_AKL:R_0805_2012Metric, symbol Device:R_US
- added R32, R33, R34, R35, R36, R37, R39, R40, R41, R42, R43, R44: 10k, Resistor_SMD:R_0805_2012Metric_Pad1.20x1.40mm_HandSolder, symbol Device:R_US
- added R38: 1M, Resistor_SMD:R_0805_2012Metric_Pad1.20x1.40mm_HandSolder, symbol Device:R_US
- added R45: 12.4k, Resistor_SMD:R_0805_2012Metric_Pad1.20x1.40mm_HandSolder, symbol Device:R_US
- added R46, R47, R49, R50: 49.9, Resistor_SMD:R_0805_2012Metric_Pad1.20x1.40mm_HandSolder, symbol Device:R_US
- added R48: 10, Resistor_SMD:R_0805_2012Metric_Pad1.20x1.40mm_HandSolder, symbol Device:R_US
- added R51, R52, R53, R54: 330, Resistor_SMD:R_0805_2012Metric_Pad1.20x1.40mm_HandSolder, symbol Device:R_US
- added U14: LP38798SD-ADJ_NOPB, bitaxe:SON50P400X400X100-13N, symbol LP38798SD-ADJ_NOPB:LP38798SD-ADJ_NOPB
- added U3: W5500, Package_QFP:LQFP-48_7x7mm_P0.5mm, symbol Interface_Ethernet:W5500
- added X1: 25Mhz, PCM_Crystal_AKL:Crystal_SMD_7050-2Pin_7.0x5.0mm, symbol PCM_Crystal_AKL:SMD7050-2
- C21, C23: value 1uF -> 18pF; footprint Capacitor_SMD:C_0402_1005Metric -> Capacitor_SMD:C_0805_2012Metric_Pad1.18x1.45mm_HandSolder; DK 587-5514-1-ND -> 4713-GMC21CG180J50NTCT-ND; PART NO (none) -> GMC21CG180J50NT; PARTNO EMK105BJ105MV-F -> (none)
- C22: footprint Capacitor_SMD:C_0402_1005Metric -> Capacitor_SMD:C_0805_2012Metric_Pad1.18x1.45mm_HandSolder; DK 587-5514-1-ND -> NMC0805X7R105K25TRPLPFCT-ND; PARTNO EMK105BJ105MV-F -> NMC0805X7R105K25TRPLPF
- C24: value 10uF -> 22uF; footprint Capacitor_SMD:C_0805_2012Metric -> Capacitor_SMD:C_1210_3225Metric_Pad1.33x2.70mm_HandSolder; DK 1276-1096-1-ND -> 490-5310-1-ND; PARTNO CL21A106KOQNNNE -> GRM32EC81E226KE15L
- C25: footprint Capacitor_SMD:C_0402_1005Metric -> Capacitor_SMD:C_1206_3216Metric_Pad1.33x1.80mm_HandSolder; DK 1276-1234-1-ND -> 4713-GMC31CG104J50NTCT-ND; PARTNO CL05A104KO5NNNC -> GMC31CG104J50NT
- R16: footprint Resistor_SMD:R_0402_1005Metric -> Resistor_SMD:R_0805_2012Metric_Pad1.20x1.40mm_HandSolder; DK 311-10KJRCT-ND -> TNP10.0KABCT-ND; PARTNO RC0402JR-0710KL -> TNPW080510K0BEEA
Connections:
- net EN: now also C22.2, R16.1, J9.1 (Pin_1); no longer C22.1, R16.2
- net GND: now also C22.1, C70.2, C71.2, C72.2, C73.2, C74.2, C75.2, C76.2, C77.1, C80.2, J10.2 (Pin_2), J10.3 (Pin_3), J10.4 (Pin_4), J11.1 (Pin_1), J8.4 (Pin_4), J8.5 (Pin_5), J9.2 (Pin_2), J9.3 (Pin_3), J9.4 (Pin_4), R31.2, R39.1, R40.1, R41.1, R42.1, R43.1, R44.1, R45.2, U14.13 (DAP), U14.5 (EN), U14.6 (GND_CP), U14.7 (GND), U3.14 (AGND), U3.16 (AGND), U3.19 (AGND), U3.29 (GND), U3.3 (AGND), U3.48 (AGND), U3.9 (AGND); no longer C22.2
- net IO0: now also J9.5 (Pin_5)
- net SCL: now also J11.3 (Pin_3)
- net SDA: now also J11.4 (Pin_4)
- net USB_D+: now also J8.3 (Pin_3)
- net USB_D-: now also J8.2 (Pin_2)
- net at U4.32 (MTCK/GPIO39/CLK_OUT3/SUBSPICS1): now also U3.34 (MISO)
- net at U4.33 (MTDO/GPIO40/CLK_OUT2): now also U3.35 (MOSI)
- net at U4.34 (MTDI/GPIO41/CLK_OUT1): now also U3.33 (SCLK)
- net at U4.35 (MTMS/GPIO42): now also R34.2, U3.32 (~{SCS})
- net 3V3 renamed +3.3V
- net +3.3V: now also R16.2, C74.1, C75.1, J11.2 (Pin_2), J4.L1, J4.L4, R32.1, R33.1, R34.1, R35.1, R36.1, R37.1, R46.1, R47.1, R48.1, R53.1, U14.10 (OUT_FB), U14.11 (OUT), U14.12 (OUT), U3.11 (AVDD), U3.15 (AVDD), U3.17 (AVDD), U3.21 (AVDD), U3.28 (VDD), U3.4 (AVDD), U3.8 (AVDD); no longer C23.1, R16.1
- net 5V: no longer names the net of C21.1
- net 5V: now also R38.1, U3.30 (XI/CLKIN), X1.2
- new net: J4.R1 (TD+), R47.2, U3.2 (TXP)
- new net: C73.1, U14.4 (CP)
- new net: R30.2, R31.1, U14.8 (FB)
- new net: R30.1, U14.9 (SET)
- new net: C76.1, J4.R4 (TCT), R48.2
- new net: C78.1, R49.1, U3.6 (RXP)
- new net: C78.2, J4.R3 (RD+)
- new net: J4.R2 (TD-), R46.2, U3.1 (TXN)
- new net: R45.1, U3.10 (EXRES1)
- new net: C71.1, U3.20 (TOCAP)
- new net: C70.1, U3.22 (1V2O)
- new net: R44.2, U3.23 (RSVD)
- new net: R51.1, U3.25 (LINKLED)
- new net: R52.1, R54.1, U3.27 (ACTLED)
- new net: C23.1, R38.2, U3.31 (XO), X1.1
- new net: R32.2, U3.36 (~{INT})
- new net: R33.2, U3.37 (~{RST})
- new net: R39.2, U3.38 (RSVD)
- new net: R40.2, U3.39 (RSVD)
- new net: R41.2, U3.40 (RSVD)
- new net: R42.2, U3.41 (RSVD)
- new net: R43.2, U3.42 (RSVD)
- new net: R37.2, U3.43 (PMODE2)
- new net: R36.2, U3.44 (PMODE1)
- new net: R35.2, U3.45 (PMODE0)
- new net: C79.1, R50.1, U3.5 (RXN)
- new net: J4.L3, R52.2
- new net: C79.2, J4.R6 (RD-)
- new net: C80.1, R49.2, R50.2
- new net: J4.L2, R51.2
- new net: J10.1 (Pin_1), R53.2
- new net +12V: C72.1, U14.1 (IN), U14.2 (IN), U14.3 (IN_CP)
- new net P,FB: C77.2, J4.R8, J4.SH
- no-connect marks 24 -> 28
Other:
- note removed: "Accessory Port"
- note removed: "ESP32 3V3 LDO"
- company: (none) -> Oconical
- title: bitaxeGamma -> bitaxeGamma 605 Kit
- moved on the sheet: J2, J3, TP10, TP11, TP5, TP6, TP7, TP9
