File: power.kicad_sch (KiCad schematic)
At the start: 40 parts, among them T1 net-tie, U2 TPS546D24ARVFR

Commit message: added files for model 605 Gamma Kit
Updated sizes for handsoldering kit, added onboard ethernet, cpu heatsink footprint, updated power supply
Parts:
- removed C1, C5, C7: 1uF, Capacitor_SMD:C_0402_1005Metric, symbol Device:C
- removed C10: 4.7uF, Capacitor_SMD:C_0402_1005Metric, symbol Device:C
- removed C11: 1000pF, Capacitor_SMD:C_0805_2012Metric, symbol Device:C
- removed C12, C8: 0.1uF, Capacitor_SMD:C_0402_1005Metric, symbol Device:C
- removed C13: 100pF, Capacitor_SMD:C_0402_1005Metric, symbol Device:C
- removed C14, C15, C16: 22uF, Capacitor_SMD:C_0805_2012Metric, symbol Device:C
- removed C17, C18, C19, C20: 100uF, Capacitor_SMD:C_1206_3216Metric, symbol Device:C
- removed C2: 10uF, Capacitor_SMD:C_0805_2012Metric, symbol Device:C
- removed C3, C4: 47uF, Capacitor_SMD:C_1210_3225Metric, symbol Device:C
- removed C6: 4700pF, Capacitor_SMD:C_0402_1005Metric, symbol Device:C
- removed C9: 2200pF, Capacitor_SMD:C_0402_1005Metric, symbol Device:C
- removed L1: 300nH, bitaxe:SLC1175-271MEC_COC, symbol Device:L
- removed R10: 68.1k, Resistor_SMD:R_0402_1005Metric, symbol Device:R_US
- removed R11: 10, Resistor_SMD:R_0402_1005Metric, symbol Device:R_US
- removed R12: 1, Resistor_SMD:R_1206_3216Metric, symbol Device:R_US
- removed R13, R14: 49.9, Resistor_SMD:R_0402_1005Metric, symbol Device:R_US
- removed R15: 10k, Resistor_SMD:R_0402_1005Metric, symbol Device:R_US
- removed R2, R3, R4, R7: ~, Resistor_SMD:R_0402_1005Metric, symbol Device:R_US
- removed R5: 14.7k, Resistor_SMD:R_0402_1005Metric, symbol Device:R_US
- removed R6: 0, Resistor_SMD:R_0402_1005Metric, symbol Device:R_US
- removed R8: 3.74k, Resistor_SMD:R_0402_1005Metric, symbol Device:R_US
- removed R9: 11.8k, Resistor_SMD:R_0402_1005Metric, symbol Device:R_US
- removed TP3, TP4: TestPoint, TestPoint:TestPoint_Pad_D1.5mm, symbol Connector:TestPoint
- removed U2: TPS546D24ARVFR, bitaxe:LQFN40-CLIP, symbol bitaxe:TPS546D24
- added C100, C101, C102, C103, C104, C99: 6800pF, symbol Device:C_Small
- added C105, C106: 1uF, symbol Device:C
- added C107, C108: .01uF, symbol Device:C
- added C109, C110: 4.7uF, symbol Device:C
- added C111, C112: 2.2uF, symbol Device:C
- added C113, C117: 0.1uF, symbol Device:C
- added C114, C118: 33pf, symbol Device:C
- added C115, C116: 1000pF, symbol Device:C
- added C119, C120: 0.1, symbol Device:C
- added C121: 100pF, symbol Device:C
- added C122, C123: 47uf, PCM_Capacitor_THT_AKL:CP_Radial_D12.5mm_P5.00mm, symbol PCM_Capacitor_AKL:CP_Radial_D12.5mm_P5.00mm
- added C124, C125, C126, C127, C128, C129, C130, C131, C132, C133, C134, C135, C144, C145, C146, C147, C148, C150: 47uF, PCM_Capacitor_THT_AKL:CP_Radial_D12.5mm_P5.00mm, symbol PCM_Capacitor_AKL:CP_Radial_D12.5mm_P5.00mm
- added C136, C137, C140, C141: 470uF, PCM_Capacitor_THT_AKL:CP_Radial_D12.5mm_P5.00mm, symbol PCM_Capacitor_AKL:CP_Radial_D12.5mm_P5.00mm
- added C138, C139: 4700pF, symbol Device:C
- added C142, C143, C149: 47000pF, symbol Device:C
- added C58, C61: .01, Capacitor_SMD:C_0805_2012Metric_Pad1.18x1.45mm_HandSolder, symbol Device:C
- added C59, C60: 1uF, Capacitor_SMD:C_0805_2012Metric_Pad1.18x1.45mm_HandSolder, symbol Device:C
- added C62, C91: 22uF, Capacitor_SMD:C_1210_3225Metric_Pad1.33x2.70mm_HandSolder, symbol Device:C
- added C87, C88: 100uF, PCM_Capacitor_THT_AKL:CP_Radial_D12.5mm_P5.00mm, symbol PCM_Capacitor_AKL:CP_Radial_D12.5mm_P5.00mm
- added C89, C92, C93, C94, C95, C96, C97, C98: 22uF, PCM_Capacitor_THT_AKL:CP_Radial_D12.5mm_P5.00mm, symbol PCM_Capacitor_AKL:CP_Radial_D12.5mm_P5.00mm
- added L2 (x2): 150nH, symbol Device:L
- added R20, R28: 47.5k, PCM_Resistor_SMD_AKL:R_0805_2012Metric, symbol Device:R_US
- added R26, R29: 15k, PCM_Resistor_SMD_AKL:R_0805_2012Metric, symbol Device:R_US
- added R27: 560k, PCM_Resistor_SMD_AKL:R_0805_2012Metric, symbol Device:R_US
- added R55, R56: 10, PCM_Resistor_SMD_AKL:R_1206_3216Metric, symbol PCM_Resistor_AKL:R_1206
- added R57, R59: 30.1k, PCM_Resistor_SMD_AKL:R_1206_3216Metric, symbol PCM_Resistor_AKL:R_1206
- added R58, R60: 7.5k, PCM_Resistor_SMD_AKL:R_1206_3216Metric, symbol PCM_Resistor_AKL:R_1206
- added R61: 10k, symbol Device:R
- added R62: 8.25k, PCM_Resistor_SMD_AKL:R_1206_3216Metric, symbol PCM_Resistor_AKL:R_1206
- added R63, R64: 10k, PCM_Resistor_SMD_AKL:R_1206_3216Metric, symbol PCM_Resistor_AKL:R_1206
- added R65: 14.7k, PCM_Resistor_SMD_AKL:R_1206_3216Metric, symbol PCM_Resistor_AKL:R_1206
- added R66: 68.1k, PCM_Resistor_SMD_AKL:R_1206_3216Metric, symbol PCM_Resistor_AKL:R_1206
- added R67, R68: 1, symbol Device:R
- added R69: 49.9, PCM_Resistor_SMD_AKL:R_1206_3216Metric, symbol PCM_Resistor_AKL:R_1206
- added R70: 49.9, symbol Device:R
- added U1, U13: TPS546D24ARVFR, bitaxe:LQFN40-CLIP, symbol PCM_bitaxe:TPS546D24
- added U11, U12: LP38798SD-ADJ_NOPB, bitaxe:SON50P400X400X100-13N, symbol LP38798SD-ADJ_NOPB:LP38798SD-ADJ_NOPB
- R1: value 8.25k -> 560k; footprint Resistor_SMD:R_0402_1005Metric -> PCM_Resistor_SMD_AKL:R_0805_2012Metric; DK 311-8.25KLRCT-ND -> 541-TNPV0805560KBEEACT-ND; PARTNO RC0402FR-078K25L -> TNPV0805560KBEEA
Connections:
- net AGND is gone; now on net GND: T1.1
- net 5V: now also C62.1, U12.10 (OUT_FB), U12.11 (OUT), U12.12 (OUT)
- net GND: now also R1.2, C100.2, C101.2, C102.2, C103.2, C104.2, C105.2, C106.2, C107.2, C108.2, C109.2, C110.2, C114.2, C118.2, C119.2, C120.2, C122.2, C123.2, C124.2, C125.2, C126.2, C127.2, C128.2, C129.2, C130.2, C131.2, C132.2, C133.2, C134.2, C135.2, C136.2, C137.2, C138.2, C139.2, C140.2, C141.2, C142.2, C143.2, C144.2, C145.2, C146.2, C147.2, C148.2, C149.2, C58.2, C59.2, C60.2, C61.2, C62.2, C87.2, C88.2, C89.2, C91.2, C92.2, C93.2, C94.2, C95.2, C96.2, C97.2, C98.2, C99.2, R26.2, R27.2, R29.2, R58.2, R60.2, R65.2, R66.2, R67.2, R68.2, U1.13 (PGND), U1.14 (PGND), U1.15 (PGND), U1.16 (PGND), U1.17 (PGND), U1.18 (PGND), U1.19 (PGND), U1.20 (PGND), U1.29 (MSEL2), U1.37 (AGND), U1.41 (PAD), U11.13 (DAP), U11.5 (EN), U11.6 (GND_CP), U11.7 (GND), U12.13 (DAP), U12.5 (EN), U12.6 (GND_CP), U12.7 (GND), U13.13 (PGND), U13.14 (PGND), U13.15 (PGND), U13.16 (PGND), U13.17 (PGND), U13.18 (PGND), U13.19 (PGND), U13.20 (PGND), U13.29 (MSEL2), U13.37 (AGND), U13.41 (PAD)
- net SCL: now also U1.3 (PMB_CLK)
- net SDA: now also U1.2 (PMB_DATA)
- net SMB_ALRT: now also U1.6 (SMB_ALRT)
- net at R1.1: now also R28.2, R29.1, U12.8 (FB)
- new net: C59.1, C60.1, U11.1 (IN), U11.2 (IN), U11.3 (IN_CP), U12.1 (IN), U12.2 (IN), U12.3 (IN_CP)
- new net: C61.1, U12.4 (CP)
- new net: R28.1, U12.9 (SET)
- new net: R63.1, U1.1 (PGD)
- new net: C113.2, C115.1, L2.1, U1.10 (SW), U1.11 (SW), U1.12 (SW), U1.8 (SW), U1.9 (SW)
- new net: C105.1, R55.2, U1.26 (AVIN)
- new net: C107.1, R57.2, R58.1, U1.27 (EN/UVLO)
- new net: R61.2, U1.34 (GOSNS)
- new net: C114.1, C118.1, U1.35 (VSHARE), U13.35 (VSHARE)
- new net: U1.38 (SYNC), U13.38 (SYNC)
- new net: U1.39 (BCX_CLK), U13.39 (BCX_CLK)
- new net: C111.2, R61.1, U1.4 (BP1V5)
- new net: U1.40 (BCX_DAT), U13.40 (BCX_DAT)
- new net: C111.1, U1.5 (DRTN)
- new net: C113.1, U1.7 (BOOT)
- new net: C119.1, C120.1, C122.1, C123.1, C124.1, C125.1, C126.1, C127.1, C128.1, C129.1, C130.1, C131.1, C132.1, C133.1, C134.1, C135.1, C136.1, C137.1, C138.1, C139.1, C140.1, C141.1, C142.1, C143.1, C144.1, C145.1, C146.1, C147.1, C148.1, C149.1, C150.1, L2.2, L2.2, R69.2
- new net: C110.1, C91.1, R64.2, U11.10 (OUT_FB), U11.11 (OUT), U11.12 (OUT), U13.28 (VDD5)
- new net: C121.1, R69.1, U13.33 (VOSNS)
- new net: C121.2, R70.1, U13.34 (GOSNS)
- new net: C112.2, R62.1, U13.4 (BP1V5)
- new net: R62.2, R65.1, U13.32 (MSEL1)
- new net: C150.2, R70.2
- new net: C108.1, R59.2, R60.1, U13.27 (EN/UVLO)
- new net: R20.2, R26.1, U11.8 (FB)
- new net: C116.2, R68.1
- new net: C115.2, R67.1
- new net: C112.1, U13.5 (DRTN)
- new net: C58.1, U11.4 (CP)
- new net: C116.1, C117.2, L2.1, U13.10 (SW), U13.11 (SW), U13.12 (SW), U13.8 (SW), U13.9 (SW)
- new net: R20.1, U11.9 (SET)
- new net: R64.1, U13.1 (PGD)
- new net: C106.1, R56.2, U13.26 (AVIN)
- new net: C117.1, U13.7 (BOOT)
- new net +12V: C100.1, C101.1, C102.1, C103.1, C104.1, C87.1, C88.1, C89.1, C92.1, C93.1, C94.1, C95.1, C96.1, C97.1, C98.1, C99.1, R55.1, R56.1, R57.1, R59.1, U1.21 (PVIN), U1.22 (PVIN), U1.23 (PVIN), U1.24 (PVIN), U1.25 (PVIN), U13.21 (PVIN), U13.22 (PVIN), U13.23 (PVIN), U13.24 (PVIN), U13.25 (PVIN)
- new net +5V: C109.1, R63.2, U1.28 (VDD5)
- no-connect marks 5 -> 0
Other:
- note added: "Input 3.3-12V 45W"
- note removed: "I2C ADDR = 0x24"
- note removed: "Input 4.5-5.5V"
- note removed: "PGD is an open drain output from the TPS546D24. Pull up to 3.3V"
- note removed: "TPS546D24A is a Buck regulator that steps 4.5-5.5V down to 1.2V @ 20A for the BM1368"
- note removed: "https://webench.ti.com/appinfo/webench/scripts/SDP.cgi?ID=3808DBEB40D18F5D"
- company: (none) -> Oconical
- title: bitaxeGamma -> bitaxeGamma 605 Kit
